File: PCB/PSU/kicad project/PSU.kicad_pcb (KiCad board)
At the start: 2 copper layers, 78 parts, among them J3 MAINS_IN, J4 Screw_Terminal_01x04, J5 T1_SEC, J6 GND_LIFT, J7 FAN1_12V, J8 FAN2_12V, SW2 V80212MS02Q, U1 LM317AT/NOPB, U2 LM337T/NOPB, U3 LD1117V33C, U5 3v3 Mornsun URB4803LD-20WR3, U6 MeanWell NID-100-5, U7 12v Mornsun URB2412LD-30WR3

Commit message: pcb rev 0
Parts:
- added H1: MountingHole_Pad, MountingHole:MountingHole_3.2mm_M3_Pad_TopBottom, F.Cu at (171.7, 86.2)
- added J2: OUT_ANLG, TerminalBlock_Phoenix:TerminalBlock_Phoenix_MKDS-1,5-4-5.08_1x04_P5.08mm_Horizontal, F.Cu at (331.8, 154.2)
- added J9: OUT_DIGI, TerminalBlock_Phoenix:TerminalBlock_Phoenix_MKDS-1,5-4-5.08_1x04_P5.08mm_Horizontal, F.Cu at (64.7, 77.9)
- added REF**: MountingHole_3.2mm_M3, MountingHole:MountingHole_3.2mm_M3, F.Cu at (379.0, 158.0)
- added REF**: Smolhaj_Scale_0.1, Symbol:Smolhaj_Scale_0.1, B.Cu at (282.9, 127.3)
- added REF**: MountingHole_3.2mm_M3, MountingHole:MountingHole_3.2mm_M3, F.Cu at (279.8, 77.2)
- added REF**: Screw_Generic_2.0x3.0mm_SilkScreen, Symbol:Screw_Generic_2.0x3.0mm_SilkScreen, F.Cu at (171.6, 80.4)
- added REF**: MountingHole_3.2mm_M3, MountingHole:MountingHole_3.2mm_M3, F.Cu at (47.8, 157.8)
- added REF**: MountingHole_3.2mm_M3, MountingHole:MountingHole_3.2mm_M3, F.Cu at (279.8, 158.0)
- added REF**: MountingHole_3.2mm_M3, MountingHole:MountingHole_3.2mm_M3, F.Cu at (379.0, 77.5)
- added REF**: MountingHole_3.2mm_M3, MountingHole:MountingHole_3.2mm_M3, F.Cu at (242.4, 123.2)
- added REF**: MountingHole_3.2mm_M3, MountingHole:MountingHole_3.2mm_M3, F.Cu at (47.8, 77.3)
- added REF**: MountingHole_3.2mm_M3, MountingHole:MountingHole_3.2mm_M3, F.Cu at (151.4, 143.2)
- added TR2: Amgis L01-6320, My Footprints:AMGIS L01-63XX, F.Cu at (203.6, 102.6)
- U6: footprint Converter_DCDC:Converter_DCDC_XP_POWER_JTDxxxxxxx_THT -> My Footprints:MeanWell NID100
- moved C5 280.1 mm to (376.9, 101.6)
- moved C6 279.7 mm to (376.9, 112.4)
- moved R10 276.2 mm to (368.0, 82.3), turned to 90 degrees
- moved U2 275.4 mm to (356.5, 102.7), turned to -90 degrees
- moved C8 274.5 mm to (378.1, 147.4), turned to 180 degrees
- moved R8 270.8 mm to (367.3, 107.0), turned to 180 degrees
- moved R6 270.5 mm to (367.3, 103.7)
- moved C2 270.4 mm to (314.1, 125.8)
- moved C4 266.7 mm to (314.2, 147.1)
- moved R9 263.3 mm to (355.5, 82.3), turned to 90 degrees
- moved C1 255.4 mm to (292.6, 125.8)
- moved C7 252.3 mm to (355.6, 132.4)
- moved C3 250.1 mm to (292.7, 147.1)
- moved D11 245.2 mm to (370.6, 77.3), turned to 180 degrees
- moved U1 243.5 mm to (323.4, 91.8), turned to -90 degrees
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Connections:
- C1 pad 2: Net-(C1-Pad2) -> Net-(D5--)
- C10 pad 1: /GND -> Net-(D5--)
- C11 pad 2: /GND -> Net-(D5--)
- C12 pad 2: /GND -> Net-(D5--)
- C13 pad 2: /GND -> Net-(D5--)
- C14 pad 2: /GND -> Net-(D5--)
- C15 pad 1: /GND -> Net-(D5--)
- C16 pad 2: Net-(D10-K) -> Net-(C16-Pad2)
- C17 pad 2: Net-(D10-K) -> Net-(C16-Pad2)
- C2 pad 1: Net-(C1-Pad2) -> Net-(D5--)
- C22 pad 1: Net-(D10-K) -> Net-(J7-Pin_2)
- C3 pad 2: Net-(C3-Pad2) -> Net-(D5--)
- C4 pad 1: Net-(C3-Pad2) -> Net-(D5--)
- C5 pad 2: /GND -> Net-(D5--)
- C6 pad 1: /GND -> Net-(D5--)
- C7 pad 2: /GND -> Net-(D5--)
- C8 pad 1: /GND -> Net-(D5--)
- C9 pad 2: /GND -> Net-(D5--)
- D5 pad 3: /GND -> Net-(D5--)
- D5 pad 4: /GND -> Net-(D5--)
- D6 pad 2: /GND -> Net-(D5--)
- D6 pad 3: /GND -> Net-(D5--)
- J5 pad 2: /GND -> Net-(D5--)
- J5 pad 3: /GND -> Net-(D5--)
- J6 pad 3: /GND -> Net-(D5--)
- J7 pad 2: Net-(D10-K) -> Net-(J7-Pin_2)
- J8 pad 2: Net-(D10-K) -> Net-(J7-Pin_2)
- L4 pad 1: Net-(D10-K) -> Net-(J7-Pin_2)
- R1 pad 2: Net-(R1-Pad2) -> Net-(D5--)
- R15 pad 2: Net-(D10-K) -> Net-(J7-Pin_2)
- R2 pad 1: Net-(R1-Pad2) -> Net-(D5--)
- R3 pad 2: /GND -> Net-(D5--)
- R4 pad 2: /GND -> Net-(D5--)
- R5 pad 2: /GND -> Net-(D5--)
- R6 pad 1: /GND -> Net-(D5--)
- U3 pad 1: /GND -> Net-(D5--)
- U7 pad 4: Net-(D10-K) -> Net-(J7-Pin_2)
Routing:
- net Net-(D10-K): track 0.00 -> 221.9 mm, vias 0 -> 35
- net Net-(J7-Pin_2): track 0.00 -> 214.6 mm, vias 0 -> 1
- net /+3V3_REF: track 0.00 -> 170.9 mm
- net Net-(D1-K): track 0.00 -> 151.7 mm
- net /+18V: track 0.00 -> 138.2 mm, vias 0 -> 1
- net Net-(U5-Vin): track 0.00 -> 137.3 mm
- net Net-(D3-A): track 0.00 -> 120.2 mm
- net /-18V: track 0.00 -> 109.8 mm, vias 0 -> 1
- net Net-(U5-Enable): track 0.00 -> 103.5 mm
- net Net-(J4-Pin_1): track 0.00 -> 89.8 mm
- net Net-(J3-Pin_2): track 0.00 -> 86.7 mm
- net Net-(U5-+VOUT): track 0.00 -> 70.0 mm
- net Net-(D5-+): track 0.00 -> 68.2 mm
- net Net-(J4-Pin_2): track 0.00 -> 66.7 mm
- net Net-(D1-A): track 0.00 -> 65.4 mm
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- added copper zone on B.Cu, net Net-(D10-K)
- added copper zone on F.Cu, net Net-(D10-K)
- added copper zone on B.Cu, net Net-(D5--)
- added copper zone on F.Cu, net Net-(D5--)
Other:
- board outline added: 341.7 x 90.9 mm
- board text added: "115"
- board text added: "230"
- board text added: "3V -18V GND +18V"
- board text added: "CHASSIS"
- board text added: "GND 3V3 Logic 5V LEDs 10V Motors"
- board text added: "GND LIFT"
- board text added: "HEATSINK"
- board text added: "L"
- board text added: "MAINS VOLTAGE"
- board text added: "N"
- board text added: "ORANGE YELLOW BLACK RED"
- board text added: "Rev 0"
- board text added: "SKD ANALOG"
- board text added: "Skylar Evelyn Denno 2026"
- board text added: "VIOLET BROWN BLUE GREY"

Commit message: pcb rev 0
Routing:
- net Net-(D5--): vias 33 -> 21
- net Net-(D10-K): vias 35 -> 9

Commit message: pcb rev 0
Other:
- board text added: "3V3 Ref -18V GND +18V"
- board text removed: "3V -18V GND +18V"
Changed lines of the file:
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@@
 		)
 		(property "Value" "MountingHole_3.2mm_M3"
-			(at 0 4.15 0)
+			(at -0.2 -3.1 0)
 			(layer "F.Fab")
 			(effects
@@
 		)
 	)
-	(gr_text "3V\n\n-18V\n\nGND\n\n+18V\n\n\n"
+	(gr_text "3V3 Ref\n\n-18V\n\nGND\n\n+18V\n\n\n"
 		(at 326.4 147.2 270)
 		(layer "F.SilkS")

Commit message: pcb rev 0
Routing:
- net Net-(D5--): track 58.9 -> 59.4 mm, vias 21 -> 22
- net Net-(D10-K): vias 9 -> 8
Changed lines of the file:
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@@
-	)
-	(via
-		(at 179.5 98)
-		(size 0.8)
-		(drill 0.5)
-		(layers "F.Cu" "B.Cu")
-		(free yes)
-		(net "Net-(D10-K)")
 	)
 	(via
@@
 	)
 	(segment
+		(start 163.535 97.990001)
+		(end 179.490001 97.990001)
+		(width 0.8)
+		(layer "F.Cu")
+		(net "Net-(D5--)")
+	)
+	(segment
 		(start 155.25905 115.15405)
 		(end 155.25905 100.896555)
@@
 	)
 	(segment
-		(start 163.535 97.990001)
-		(end 178.974999 97.990001)
-		(width 0.8)
-		(layer "F.Cu")
-		(net "Net-(D5--)")
-	)
-	(segment
 		(start 236.52 94.3)
 		(end 237.145 94.3)
@@
 		(net "Net-(D5--)")
 	)
+	(segment
+		(start 179.490001 97.990001)
+		(end 179.5 98)
+		(width 0.8)
+		(layer "F.Cu")
+		(net "Net-(D5--)")
+	)
 	(via
 		(at 348.4 92)
@@
 		(size 0.8)
 		(drill 0.5)
+		(layers "F.Cu" "B.Cu")
+		(free yes)
+		(net "Net-(D5--)")
+	)
+	(via
+		(at 179.5 98)
+		(size 0.8)
+		(drill 0.5)

Commit message: pcb rev 0
Parts:
- added J10: SMPS_IN, TerminalBlock_Phoenix:TerminalBlock_Phoenix_MKDS-1,5-2-5.08_1x02_P5.08mm_Horizontal, F.Cu at (143.1, 153.4)
- moved J3 4.64 mm to (180.0, 153.4), turned to 0 degrees
Routing:
- net Net-(J10-Pin_2): track 15.6 -> 99.1 mm
- net Net-(J10-Pin_1): track 7.39 -> 77.8 mm
- net Net-(J3-Pin_2): track 86.7 -> 78.7 mm
- net Net-(J3-Pin_1): track 16.1 -> 19.0 mm
- net Net-(D5--): vias 22 -> 23
Other:
- board text added: "+15V"

Commit message: rev 0.1 4 layer
Parts:
- removed the REF** at (282.9, 127.3)
- added REF**: Screw_Generic_2.0x3.0mm_SilkScreen, Symbol:Screw_Generic_2.0x3.0mm_SilkScreen, F.Cu at (373.3, 156.6)
- added REF**: Screw_Generic_2.0x3.0mm_SilkScreen, Symbol:Screw_Generic_2.0x3.0mm_SilkScreen, F.Cu at (146.7, 135.0)
- added REF**: Screw_Generic_2.0x3.0mm_SilkScreen, Symbol:Screw_Generic_2.0x3.0mm_SilkScreen, F.Cu at (380.0, 82.9)
- added REF**: Screw_Generic_2.0x3.0mm_SilkScreen, Symbol:Screw_Generic_2.0x3.0mm_SilkScreen, F.Cu at (284.5, 155.8)
- added REF**: Screw_Generic_2.0x3.0mm_SilkScreen, Symbol:Screw_Generic_2.0x3.0mm_SilkScreen, F.Cu at (240.0, 118.3)
- added REF**: Screw_Generic_2.0x3.0mm_SilkScreen, Symbol:Screw_Generic_2.0x3.0mm_SilkScreen, F.Cu at (45.1, 82.3)
- added REF**: Screw_Generic_2.0x3.0mm_SilkScreen, Symbol:Screw_Generic_2.0x3.0mm_SilkScreen, F.Cu at (52.0, 155.8)
- added REF**: Screw_Generic_2.0x3.0mm_SilkScreen, Symbol:Screw_Generic_2.0x3.0mm_SilkScreen, F.Cu at (274.3, 77.5)
- moved REF** 4.08 mm to (149.3, 139.7)
- moved REF** 1.43 mm to (377.6, 77.2)
- moved REF** 1.41 mm to (377.6, 158.2)
- moved REF** 0.45 mm to (47.6, 158.2)
- moved REF** 0.25 mm to (279.6, 158.2)
- moved REF** 0.22 mm to (47.6, 77.2)
- moved REF** 0.16 mm to (279.6, 77.2)
Routing:
- net Net-(D10-K): vias 8 -> 10
- added copper zone on In1.Cu, net Net-(D10-K)
- added copper zone on In2.Cu, net Net-(D10-K)
- added copper zone on In1.Cu, net Net-(D5--)
- added copper zone on In2.Cu, net Net-(D5--)
Other:
- board size 341.7 x 90.9 mm -> 340 x 91 mm
- copper layers 2 -> 4
- board text added: "Rev 0.1"
- board text added: "TR1 Secondary"
- board text removed: "Rev 0"

Commit message: quick update / fix
Parts:
- added REF**: Screw_Generic_2.0x3.0mm_SilkScreen, Symbol:Screw_Generic_2.0x3.0mm_SilkScreen, F.Cu at (175.5, 81.8)
- added REF**: MountingHole_4.3mm_M4, MountingHole:MountingHole_4.3mm_M4, F.Cu at (171.7, 77.9)
- REF** (x8): value MountingHole_3.2mm_M3 -> MountingHole_4.3mm_M4; footprint MountingHole:MountingHole_3.2mm_M3 -> MountingHole:MountingHole_4.3mm_M4
- U5: value 3v3 Mornsun URB4803LD-20WR3 -> 3v3 Mornsun URB2403LD-20WR3
- U7: value 12v Mornsun URB2412LD-30WR3 -> 12v Mornsun URB2412LD-50WR3; footprint Converter_DCDC:Converter_DCDC_XP_POWER_JTDxxxxxxx_THT -> My Footprints:urb 50w dc-dc
- moved REF** 3.92 mm to (168.0, 81.9)
Connections:
- U5 pad 2: Net-(U5-Vin) -> Net-(D10-K)
- U5 pad 3: Net-(D10-K) -> Net-(U5-Vin)
- U5 pad 5: Net-(D10-K) -> unconnected-(U5-Trim-Pad5)
- U5 pad 6: unconnected-(U5-Trim-Pad6) -> Net-(D10-K)
- U7 pad 2: Net-(U5-Vin) -> Net-(D10-K)
- U7 pad 3: Net-(D10-K) -> Net-(U5-Vin)
Routing:
- net Net-(U5-Vin): track 137.5 -> 157.1 mm
- net Net-(U7-Trim): track 22.9 -> 11.5 mm, vias 1 -> 0
- net Net-(J7-Pin_2): track 214.6 -> 212.6 mm
- net Net-(U5-Enable): track 103.5 -> 101.5 mm
- net Net-(D10-K): track 221.9 -> 223.7 mm, vias 10 -> 8

Commit message: quick update / fix
Routing:
- net Net-(J7-Pin_2): track 212.6 -> 208.5 mm
Changed lines of the file:
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@@
-	)
-	(segment
-		(start 131.97 157.04)
-		(end 136.25 161.32)
-		(width 1.7)
-		(layer "F.Cu")
-		(net "Net-(J7-Pin_2)")
 	)
 	(segment
@@
 	(segment
 		(start 136.31 161.38)
-		(end 62.425 161.38)
+		(end 129.6 161.38)
 		(width 0.8)
 		(layer "F.Cu")
@@
 		(start 161.835 158.33)
 		(end 161.835 158.69)
+		(width 0.8)
+		(layer "F.Cu")
+		(net "Net-(J7-Pin_2)")
+	)
+	(segment
+		(start 129.6 161.38)
+		(end 129.635 161.345)
+		(width 0.8)
+		(layer "F.Cu")
+		(net "Net-(J7-Pin_2)")
+	)
+	(segment
+		(start 129.635 161.345)
+		(end 129.635 157.04)
 		(width 0.8)
 		(layer "F.Cu")
@@
 	)
 	(segment
-		(start 129.635 157.04)
-		(end 131.97 157.04)
-		(width 1.7)
+		(start 159.145 161.38)
+		(end 136.31 161.38)
+		(width 0.8)
 		(layer "F.Cu")
 		(net "Net-(J7-Pin_2)")
 	)
 	(segment
-		(start 159.145 161.38)
-		(end 136.31 161.38)
+		(start 129.6 161.38)
+		(end 62.425 161.38)
 		(width 0.8)
 		(layer "F.Cu")
