File: PCB/PSU/kicad project/PSU.kicad_pcb (KiCad board)
At the start: 4 copper layers, 340 x 91 mm, 102 parts, among them J10 SMPS_IN, J2 OUT_ANLG, J3 MAINS_IN, J4 Screw_Terminal_01x04, J5 T1_SEC, J6 GND_LIFT, J7 FAN1_12V, J8 FAN2_12V, J9 OUT_DIGI, SW2 V80212MS02Q, U1 LM317AT/NOPB, U2 LM337T/NOPB, U3 LD1117V33C, U5 3v3 Mornsun URB2403LD-20WR3, U6 MeanWell NID-100-5, U7 12v Mornsun URB2412LD-50WR3

Commit message: did some stuff lol
Parts:
- TR2: value Amgis L01-6320 -> Amgis L01-6330
Routing:
- net /+5V_LEDS: track 58.9 -> 64.2 mm
- net Net-(D10-K): vias 8 -> 7
Changed lines of the file:
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@@
 		(sheetname "/")
 		(sheetfile "PSU.kicad_sch")
-		(units
-			(unit
-				(name "A")
-				(pins "4" "2" "3" "1")
-			)
-		)
 		(attr through_hole)
 		(duplicate_pad_numbers_are_jumpers no)
 		(fp_line
-			(start -3.8 -3.1)
-			(end -2.5 -3.1)
+			(start 28.86 -3.16)
+			(end 27.56 -3.16)
 			(stroke
 				(width 0.12)
@@
 		)
 		(fp_line
-			(start 0.45 -2.9)
-			(end 0.45 -1.5)
-			(stroke
-				(width 0.12)
-				(type solid)
-			)
-			(layer "F.SilkS")
-		)
-		(fp_line
 			(start -3.6 -2.9)
 			(end 28.6 -2.9)
@@
 		)
 		(fp_line
-			(start -3.8 -1.7)
-			(end -3.8 -3.1)
+			(start 28.86 -1.76)
+			(end 28.86 -3.16)
 			(stroke
 				(width 0.12)
@@
 		)
 		(fp_line
-			(start 0.45 2.9)
-			(end 0.45 1.5)
-			(stroke
-				(width 0.12)
-				(type solid)
-			)
-			(layer "F.SilkS")
-		)
-		(fp_line
 			(start -3.6 2.9)
 			(end -3.6 -2.9)
@@
 		(fp_line
 			(start 28.5 -2.8)
-			(end -2.5 -2.8)
-			(stroke
-				(width 0.12)
-				(type solid)
-			)
-			(layer "F.Fab")
-		)
-		(fp_line
-			(start 0.45 -2.8)
-			(end 0.45 2.8)
-			(stroke
-				(width 0.12)
-				(type solid)
-			)
-			(layer "F.Fab")
-		)
-		(fp_line
-			(start -2.5 -2.8)
-			(end -3.5 -1.7)
+			(end -3.49 -2.8)
 			(stroke
 				(width 0.12)
@@
 		)
 		(fp_line
-			(start -3.5 -1.7)
+			(start -3.5 -2.8)
 			(end -3.5 2.8)
 			(stroke
@@
 			)
 		)
-		(pad "1" thru_hole circle
+		(pad "1" thru_hole rect
 			(at 25 0 90)
 			(size 2.5 2.5)
@@
 			(pintype "passive")
 		)
-		(pad "4" thru_hole rect
+		(pad "4" thru_hole circle
 			(at 0 0 90)
 			(size 2.5 2.5)
@@
 			)
 		)
-		(property "Value" "Amgis L01-6320"
+		(property "Value" "Amgis L01-6330"
 			(at 0.045 3.63 0)
 			(unlocked yes)
@@
 		(sheetname "/")
 		(sheetfile "PSU.kicad_sch")
-		(units
-			(unit
-				(name "A")
-				(pins "4" "2" "3" "1")
-			)
-		)
 		(attr through_hole)
 		(duplicate_pad_numbers_are_jumpers no)
 		(fp_line
-			(start -3.8 -3.1)
-			(end -2.5 -3.1)
+			(start 28.86 -3.16)
+			(end 27.56 -3.16)
 			(stroke
 				(width 0.12)
@@
 		)
 		(fp_line
-			(start 0.45 -2.9)
-			(end 0.45 -1.5)
-			(stroke
-				(width 0.12)
-				(type solid)
-			)
-			(layer "F.SilkS")
-		)
-		(fp_line
 			(start -3.6 -2.9)
 			(end 28.6 -2.9)
@@
 		)
 		(fp_line
-			(start -3.8 -1.7)
-			(end -3.8 -3.1)
+			(start 28.86 -1.76)
+			(end 28.86 -3.16)
 			(stroke
 				(width 0.12)
@@
 		)
 		(fp_line
-			(start 0.45 2.9)
-			(end 0.45 1.5)
-			(stroke
-				(width 0.12)
-				(type solid)
-			)
-			(layer "F.SilkS")
-		)
-		(fp_line
 			(start -3.6 2.9)
 			(end -3.6 -2.9)
@@
 		(fp_line
 			(start 28.5 -2.8)
-			(end -2.5 -2.8)
-			(stroke
-				(width 0.12)
-				(type solid)
-			)
-			(layer "F.Fab")
-		)
-		(fp_line
-			(start 0.45 -2.8)
-			(end 0.45 2.8)
+			(end -3.49 -2.8)
 			(stroke
 				(width 0.12)
@@
 		)
 		(fp_line
-			(start -2.5 -2.8)
-			(end -3.5 -1.7)
-			(stroke
-				(width 0.12)
-				(type solid)
-			)
-			(layer "F.Fab")
-		)
-		(fp_line
-			(start -3.5 -1.7)
+			(start -3.5 -2.8)
 			(end -3.5 2.8)
 			(stroke
@@
 			)
 		)
-		(pad "1" thru_hole circle
+		(pad "1" thru_hole rect
 			(at 25 0 90)
 			(size 2.5 2.5)
@@
 			(pintype "passive")
 		)
-		(pad "4" thru_hole rect
+		(pad "4" thru_hole circle
 			(at 0 0 90)
 			(size 2.5 2.5)
@@
 		(start 61.560001 137.980002)
 		(end 61.560001 130.887501)
-		(width 1.7)
+		(width 2.5)
 		(layer "F.Cu")
 		(net "Net-(U5-Enable)")
@@
 		(start 82.635002 137.980002)
 		(end 83.915 139.26)
-		(width 1.7)
+		(width 0.8)
 		(layer "F.Cu")
 		(net "Net-(U5-Enable)")
@@
 		(start 83.915 139.26)
 		(end 88.94 139.26)
-		(width 1.7)
+		(width 0.8)
 		(layer "F.Cu")
 		(net "Net-(U5-Enable)")
@@
 		(start 61.560001 137.980002)
 		(end 82.635002 137.980002)
-		(width 1.7)
+		(width 0.8)
 		(layer "F.Cu")
 		(net "Net-(U5-Enable)")
@@
 		(start 88.94 139.26)
 		(end 118.575 109.625)
-		(width 1.7)
+		(width 0.8)
 		(layer "F.Cu")
 		(net "Net-(U5-Enable)")
@@
 		(start 51.48 143.11)
 		(end 56.609998 137.980002)
-		(width 1.7)
+		(width 2.5)
 		(layer "B.Cu")
 		(net "Net-(U5-Enable)")
@@
 		(start 56.609998 137.980002)
 		(end 61.560001 137.980002)
-		(width 1.7)
+		(width 2.5)
 		(layer "B.Cu")
 		(net "Net-(U5-Enable)")
@@
 		(start 47.735 148.19)
 		(end 47.735 150.729999)
-		(width 1.7)
+		(width 2.5)
 		(layer "B.Cu")
 		(net "Net-(U5-Enable)")
@@
 		(start 47.735 143.11)
 		(end 47.735 145.65)
-		(width 1.7)
+		(width 2.5)
 		(layer "B.Cu")
 		(net "Net-(U5-Enable)")
@@
 		(start 47.735 143.11)
 		(end 51.48 143.11)
-		(width 1.7)
+		(width 2.5)
 		(layer "B.Cu")
 		(net "Net-(U5-Enable)")
@@
 		(start 47.735 145.65)
 		(end 47.735 148.19)
-		(width 1.7)
+		(width 2.5)
 		(layer "B.Cu")
 		(net "Net-(U5-Enable)")
@@
 	)
 	(via
-		(at 54 113.5)
-		(size 0.8)
-		(drill 0.5)
-		(layers "F.Cu" "B.Cu")
-		(free yes)
-		(net "Net-(D10-K)")
-	)
-	(via
 		(at 73.5 110)
 		(size 0.8)
@@
 		(start 60.735 92.065)
 		(end 64.71 88.09)
-		(width 1.7)
-		(layer "F.Cu")
-		(net "/+5V_LEDS")
-	)
-	(segment
-		(start 58.335 116.8475)
-		(end 58.335 108.48)
-		(width 1.7)
+		(width 2.5)
 		(layer "F.Cu")
 		(net "/+5V_LEDS")
@@
 		(start 61.06 119.5725)
 		(end 58.335 116.8475)
-		(width 1.7)
+		(width 2.5)
 		(layer "F.Cu")
 		(net "/+5V_LEDS")
@@
 		(start 60.735 100.075)
 		(end 60.735 92.065)
-		(width 1.7)
+		(width 2.5)
+		(layer "F.Cu")
+		(net "/+5V_LEDS")
+	)
+	(segment
+		(start 58.335 116.835)
+		(end 51.9 110.4)
+		(width 2.5)
+		(layer "F.Cu")
+		(net "/+5V_LEDS")
+	)
+	(segment
+		(start 58.335 116.8475)
+		(end 58.335 116.835)
+		(width 2.5)
 		(layer "F.Cu")
 		(net "/+5V_LEDS")
 	)
 	(via
-		(at 58.335 108.48)
-		(size 0.8)
-		(drill 0.5)
+		(at 51.9 110.4)
+		(size 0.6)
+		(drill 0.3)
 		(layers "F.Cu" "B.Cu")
 		(net "/+5V_LEDS")
 	)
 	(segment
-		(start 58.335 108.48)
-		(end 58.335 102.475)
-		(width 1.7)
+		(start 51.9 110.4)
+		(end 51.9 108.91)
+		(width 2.5)
 		(layer "B.Cu")
 		(net "/+5V_LEDS")
 	)
 	(segment
-		(start 58.335 102.475)
+		(start 51.9 108.91)
 		(end 60.735 100.075)
-		(width 1.7)
+		(width 2.5)
 		(layer "B.Cu")
 		(net "/+5V_LEDS")
