File: PCB/PSU/kicad project/PSU.kicad_sch (KiCad schematic)
At the start: 82 parts, among them J1 IEC_60320_C14_Receptacle, J10 FAN2_10V, J2 GND_LIFT, J3 MAINS_IN, J4 Screw_Terminal_01x04, J5 T1_SEC, J6 OUT, J9 FAN1_10V, SW1 POWER_FRNT_PNL, SW2 V80212MS02Q, U1 LM317_TO-220, U2 LM337_TO220, U3 LD1117V33, U4 MeanWell RS-75-15, U5 3v3 Mornsun URB4803LD-20WR3, U6 MeanWell_NID100, U7 12v Mornsun URB2412LD-30WR3

Commit message: cleanup + prep for pcb design
Parts:
- removed C16, C18, C20: 10u, symbol Device:C
- removed C17, C19, C21: 100n, symbol Device:C
- removed FB1: FerriteBead, Inductor_SMD:L_1206_3216Metric, symbol Device:FerriteBead
- removed R12, R3, R4: 2.7k, symbol Device:R_US
- removed R5, R6: 1, symbol Device:R_US
- added C16, C18, C20, C22: 1000u, Capacitor_THT:CP_Radial_D12.5mm_P5.00mm, symbol Device:C_Polarized
- added C17, C19, C21, C23: 470u, Capacitor_THT:CP_Radial_D10.0mm_P5.00mm, symbol Device:C_Polarized
- added L3, L4: 4.7u, Inductor_SMD:L_Vishay_IHLP-5050, symbol Device:L
- added M1, M2: Fan, symbol Motor:Fan
- added R15: 56k, Resistor_SMD:R_1206_3216Metric, symbol Device:R_US
- added R16, R17, R18, R19: 0.33R, Resistor_THT:R_Axial_DIN0207_L6.3mm_D2.5mm_P10.16mm_Horizontal, symbol Device:R_US
- C10, C14, C9: footprint (none) -> Capacitor_SMD:C_1206_3216Metric; LCSC (none) -> C1945
- C13, C7, C8: footprint (none) -> Capacitor_THT:C_Rect_L24.0mm_W12.6mm_P22.50mm_MKT
- C15: footprint (none) -> Capacitor_SMD:C_1206_3216Metric; LCSC C328801 -> C55077
- C5, C6: footprint (none) -> Capacitor_SMD:CP_Elec_6.3x5.4; symbol Device:C -> Device:C_Polarized; LCSC C328801 -> C14162
- D10, D11, D12, D13, D14, D15: footprint (none) -> LED_THT:LED_Rectangular_W3.9mm_H1.8mm; PURC_LINK (none) -> https://www.digikey.com/en/products/detail/kingbright/WP113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; now left out of the parts list
- D7, D8, D9: footprint Diode_THT:D_DO-35_SOD27_P7.62mm_Horizontal -> Diode_SMD:D_SOD-123; LCSC (none) -> C2099
- F1: PURC_LINK (none) -> https://www.digikey.com/en/products/detail/littelfuse-inc/0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
- HS1, HS2, HS3: PURC_LINK (none) -> https://www.digikey.com/en/products/detail/same-sky-formerl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
- J1: PURC_LINK (none) -> https://www.digikey.com/en/products/detail/qualtek/723W-X2-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
- J2: renamed from J6; PURC_LINK (none) -> https://www.digikey.com/en/products/detail/same-sky-formerl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; now left out of the parts list
- J3: LCSC (none) -> C5443539
- J4: LCSC (none) -> C5443561
- J5: footprint TerminalBlock_Phoenix:TerminalBlock_Phoenix_MKDS-1,5-3-5.08_1x03_P5.08mm_Horizontal -> TerminalBlock_Phoenix:TerminalBlock_Phoenix_MKDS-1,5-4_1x04_P5.00mm_Horizontal; symbol Connector:Screw_Terminal_01x03 -> Connector:Screw_Terminal_01x04; LCSC (none) -> C5443561
- J7: renamed from J9; value FAN1_10V -> FAN1_12V
- J8: renamed from J10; value FAN2_10V -> FAN2_12V
- L1, L2: value 10u -> 4.7u; footprint Inductor_SMD:L_SXN_SMDRI125 -> Inductor_SMD:L_Vishay_IHLP-5050; LCSC C9904 -> C845092
- R1, R2: value 2.7k -> 1k; footprint (none) -> Resistor_THT:R_Axial_DIN0414_L11.9mm_D4.5mm_P20.32mm_Horizontal; LCSC (none) -> C5200473
- R10: renamed from R15; footprint (none) -> Resistor_SMD:R_1206_3216Metric; LCSC (none) -> C26030
- R11: renamed from R16; footprint (none) -> Resistor_SMD:R_1206_3216Metric; LCSC (none) -> C49286685
- R12: renamed from R17; footprint (none) -> Resistor_SMD:R_1206_3216Metric; LCSC (none) -> C49286685
- R13: renamed from R18; footprint (none) -> Resistor_SMD:R_1206_3216Metric; LCSC (none) -> C49330184
- R14: renamed from R19; footprint (none) -> Resistor_SMD:R_1206_3216Metric; LCSC (none) -> C17984
- R3: renamed from R11; value 2.7k -> 1k; footprint (none) -> Resistor_THT:R_Axial_DIN0414_L11.9mm_D4.5mm_P20.32mm_Horizontal; LCSC (none) -> C5200473
- R4: renamed from R13; footprint (none) -> Resistor_SMD:R_0805_2012Metric; LCSC (none) -> C340448
- R5: renamed from R7; footprint (none) -> Resistor_SMD:R_1206_3216Metric; LCSC (none) -> C702850
- R6: renamed from R8; footprint (none) -> Resistor_SMD:R_1206_3216Metric; LCSC (none) -> C702850
- R7: renamed from R9; footprint (none) -> Resistor_SMD:R_1206_3216Metric; LCSC (none) -> C497314
- R8: renamed from R10; footprint (none) -> Resistor_SMD:R_1206_3216Metric; LCSC (none) -> C497314
- R9: renamed from R14; footprint (none) -> Resistor_SMD:R_1206_3216Metric; LCSC (none) -> C26030
- SW1: PURC_LINK (none) -> https://www.digikey.com/en/products/detail/zf-electronics/W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
- SW2: LCSC C315812 -> (none); PURC_LINK (none) -> https://www.digikey.com/en/products/detail/c-k/S202121MS02Q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; now left out of the parts list
- TH1: value NTC 5D-7 -> MF72-010D9; footprint (none) -> Capacitor_THT:C_Disc_D12.5mm_W5.0mm_P7.50mm; LCSC C5385 -> (none); PURC_LINK (none) -> https://www.digikey.com/en/products/detail/cantherm/MF72-01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
- TR1: value VTX-146-050-218 -> VTX-146-060-218; PURC_LINK (none) -> https://www.newark.com/vigortronix/vtx-146-060-218/60va-tor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
- TR2: footprint (none) -> My Footprints:Untitled; PURC_LINK (none) -> https://www.digikey.com/en/products/detail/amgis-llc/L01-63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
- U1: value LM317_TO-220 -> LM317AT/NOPB; Field5 (none) -> C94659
- U2: value LM337_TO220 -> LM337T/NOPB; LCSC (none) -> C2869423
- U3: value LD1117V33 -> LD1117V33C; LCSC (none) -> C672117
- U4: value MeanWell RS-75-15 -> MeanWell RS-100-15; footprint Converter_ACDC:Converter_ACDC_MeanWell_IRM-60-xx_THT -> (none); PURC_LINK (none) -> https://www.digikey.com/en/products/detail/mean-well-usa-in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; now left out of the parts list
- U5, U7: PURC_LINK (none) -> https://www.digikey.com/en/products/detail/mornsun-america-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; now left out of the parts list
- U6: value MeanWell_NID100 -> MeanWell NID-100-5; footprint My Footprints:MeanWell NID100 -> Converter_DCDC:Converter_DCDC_XP_POWER_JTDxxxxxxx_THT; PURC_LINK (none) -> https://www.digikey.com/en/products/detail/mean-well-usa-in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; now left out of the parts list
- renumbered J2 to J6
Connections:
- net +10V_MOTORS: now also L4.2, R19.1; no longer J7.1 (Pin_1), J8.1 (Pin_1), U7.4 (+VOUT)
- net +3V3_LOGIC: now also L2.2, R17.1
- net +5V_LEDS: now also L3.2, R18.1; no longer U5.1 (Enable), U6.1 (Vout), U6.2 (Vout), U6.3 (Vout), U6.4 (Vout), U7.1 (Enable)
- net GND: now also J5.3 (Pin_3); no longer C1.2, C2.1, D10.1 (K), D11.1 (K), D12.1 (K), D13.1 (K), D14.1 (K), D15.1 (K), J2.8, R1.2, R2.1
- net at J4.1 (Pin_1), TH1.2, TR2.1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: now also SW2.1a; no longer SW2.1 (A)
- net at J4.2 (Pin_2), TR2.2: now also SW2.2; no longer SW2.5 (B)
- net at J3.2 (Pin_2), J4.4 (Pin_4), TR2.4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: now also SW2.2a; no longer SW2.6 (C)
- net at C2.2, D3.2 (A), D4.2 (A)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: now also C4.2, D8.2 (A), U2.2 (VI); no longer L2.2
- net at U5.2 (Vin), U6.10 (Vin), U6.9 (Vin)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: now also L1.2, R16.1; no longer U4.3 (+Vout)
- net at C15.2, D6.1 (+), D6.4 (-)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: now also D10.1 (K), D11.1 (K), D12.1 (K), D13.1 (K), D14.1 (K), D15.1 (K), J7.1 (Pin_1), J8.1 (Pin_1), U7.4 (+VOUT), C16.2, C17.2, C22.1, C22.2, C23.2, L4.1, R15.2
- net at C4.1: now also C3.2
- net at C1.1, D1.1 (K), D2.1 (K)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: now also C3.1, D7.1 (K), U1.3 (VI); no longer L1.1
- net at D2.2 (A), D3.1 (K): now also J5.4 (Pin_4); no longer J5.3 (Pin_3)
- net at U5.4 (+VOUT): now also L2.1, C18.1
- net at TR1.6: no longer TR1.7
- net at U7.6 (Trim): now also R15.1
- new net: C21.1, R18.2
- new net: C20.2, C21.2
- new net: J4.3 (Pin_3), SW2.1, SW2.1b, SW2.2b, TR2.3
- new net: R1.2, R2.1
- new net: C16.1, L1.1, U4.3 (+Vout)
- new net: C20.1, L3.1, U5.1 (Enable), U6.1 (Vout), U6.2 (Vout), U6.3 (Vout), U6.4 (Vout), U7.1 (Enable)
- new net: C1.2, C2.1
- new net: C23.1, R19.2
- new net: C18.2, C19.2
- new net: C19.1, R17.2
- new net: C17.1, R16.2
Other:
- note added: "COMPONENT NOTES: R1, R2, R3, (discharges big filter caps) use at least 1W at least Resistors. For all other resistors, use 1/4W. All resistors are metal film, 1% or better tolerance. All screw terminals (J3, J4. J5) are the Phoenix Contact MKDS 1,5 series, 5.08mm pin pitch. Pin headers (J2, J9, J10) are standard 2.54mm pin pitch male pin headers. Regulators (U1, U2, U3) are all TO-220 3 pin packa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"
- note added: "Indicator LEDs"
- note added: "Short 2&3 for direct ground"
- note removed: "COMPONENT NOTES: R1, R2, R3, R4, R11, R12: use 1W Resistors. For all other resistors, use 1/4W. All resistors are metal film 1% or better tolerance. All screw terminals (J3, J4. J5, J7, J8) are the Phoenix Contact MKDS 1,5 series, 5.08mm pin pitch. Pin headers (J2, J9, J10) are standard 2.54mm pin pitch male pin headers. Polarized capacitors (C1, C2, C3, C4, C11, C12) are electrolytics - at least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"
- note removed: "Short 1&2 for ground lift Short 2&3 for direct ground"
- moved on the sheet: C1, C11, C12, C2, C3, C4, J7, J8, R1, R2, R3, U5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

Commit message: pcb rev 0
Parts:
- removed J2: OUT, TerminalBlock_Phoenix:TerminalBlock_Phoenix_MKDS-1,5-8-5.08_1x08_P5.08mm_Horizontal, symbol Connector:DIN-8
- added H1: MountingHole_Pad, MountingHole:MountingHole_3.2mm_M3_Pad_TopBottom, symbol Mechanical:MountingHole_Pad
- added J2: OUT_ANLG, TerminalBlock_Phoenix:TerminalBlock_Phoenix_MKDS-1,5-4-5.08_1x04_P5.08mm_Horizontal, symbol Connector:Screw_Terminal_01x04
- added J9: OUT_DIGI, TerminalBlock_Phoenix:TerminalBlock_Phoenix_MKDS-1,5-4-5.08_1x04_P5.08mm_Horizontal, symbol Connector:Screw_Terminal_01x04
- TH1: now left out of the parts list
- TR2: footprint My Footprints:Untitled -> My Footprints:AMGIS L01-63XX
- U1: Field5 C94659 -> (none); LCSC (none) -> C94659
- U6: footprint Converter_DCDC:Converter_DCDC_XP_POWER_JTDxxxxxxx_THT -> My Footprints:MeanWell NID100
Connections:
- net GND is gone; now on an unnamed net: C10.1, C11.2, C12.2, C13.2, C14.2, C15.1, C5.2, C6.1, C7.2, C8.1, C9.2, D5.3, D5.4 (-), D6.2, D6.3, J5.2 (Pin_2), J5.3 (Pin_3), J6.3 (Pin_3), R3.2, R4.2, R5.2, R6.1, TR2.5, TR2.7, U3.1 (GND)
- net +10V_MOTORS: now also J9.4 (Pin_4)
- net +18V: now also J2.1 (Pin_1)
- net +3V3_LOGIC: now also J9.2 (Pin_2)
- net +3V3_REF: now also J2.4 (Pin_4)
- net +5V_LEDS: now also J9.3 (Pin_3)
- net -18V: now also J2.3 (Pin_3)
- net at J4.1 (Pin_1), SW2.1a, TH1.2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: no longer U4.1 (AC/L)
- net at J3.2 (Pin_2), J4.4 (Pin_4), SW2.2a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: no longer U4.2 (AC/N)
- net at C15.2, C22.2, C23.2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: now also H1.1, J9.1 (Pin_1); no longer C16.2, C17.2, C22.1, J7.2 (Pin_2), J8.2 (Pin_2), L4.1, R15.2, U4.4 (-Vout), U7.4 (+VOUT)
- net at R1.2, R2.1: now also C1.2, C2.1, C3.2, C4.1, J2.2 (Pin_2)
- new net: C16.2, C17.2, U4.4 (-Vout)
- new net: C22.1, J7.2 (Pin_2), J8.2 (Pin_2), L4.1, R15.2, U7.4 (+VOUT)
Other:
- note added: "COMPONENT NOTES: R1, R2, R3, (discharges big filter caps) use at least 1W at least Resistors. For all other resistors, use 1/4W. All resistors are metal film, 1% or better tolerance. All screw terminals (J2, J3, J4. J5, J9, J10) are the Phoenix Contact MKDS 1,5 series, 5.08mm pin pitch. Pin headers (J2, J9, J10) are standard 2.54mm pin pitch male pin headers. Regulators (U1, U2, U3) are all TO-22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"
- note removed: "COMPONENT NOTES: R1, R2, R3, (discharges big filter caps) use at least 1W at least Resistors. For all other resistors, use 1/4W. All resistors are metal film, 1% or better tolerance. All screw terminals (J3, J4. J5) are the Phoenix Contact MKDS 1,5 series, 5.08mm pin pitch. Pin headers (J2, J9, J10) are standard 2.54mm pin pitch male pin headers. Regulators (U1, U2, U3) are all TO-220 3 pin packa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"

Commit message: pcb rev 0
Parts:
- added J10: SMPS_IN, TerminalBlock_Phoenix:TerminalBlock_Phoenix_MKDS-1,5-2-5.08_1x02_P5.08mm_Horizontal, symbol Connector:Screw_Terminal_01x02
Connections:
- net at C16.1, L1.1: now also J10.1 (Pin_1); no longer U4.3 (+Vout)
- net at C16.2, C17.2: now also J10.2 (Pin_2); no longer U4.4 (-Vout)
Changed lines of the file:
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@@
 	(paper "A3")
 	(arc
+		(start 165.1 138.43)
+		(mid 168.538 137.7499)
+		(end 171.45 139.7)
+		(stroke
+			(width 0)
+			(type default)
+		)
+		(fill
+			(type none)
+		)
+	)
+	(arc
 		(start 76.2004 90.1851)
 		(mid 114.7355 105.3467)
@@
 	)
 	(arc
+		(start 165.1 143.51)
+		(mid 168.012 141.5599)
+		(end 171.45 142.24)
+		(stroke
+			(width 0)
+			(type default)
+		)
+		(fill
+			(type none)
+		)
+	)
+	(arc
 		(start 171.45 54.61)
 		(mid 182.508 50.7736)
@@
 	)
 	(junction
-		(at 184.15 138.43)
-		(diameter 0)
-		(color 0 0 0 0)
-	)
-	(junction
 		(at 119.38 48.26)
 		(diameter 0)
@@
 	)
 	(junction
+		(at 184.15 139.7)
+		(diameter 0)
+		(color 0 0 0 0)
+	)
+	(junction
 		(at 295.91 100.33)
 		(diameter 0)
@@
 	(wire
 		(pts
+			(xy 176.53 139.7) (xy 184.15 139.7)
+		)
+		(stroke
+			(width 0)
+			(type default)
+		)
+	)
+	(wire
+		(pts
 			(xy 290.83 133.35) (xy 293.37 133.35)
 		)
@@
 	(wire
 		(pts
+			(xy 151.13 143.51) (xy 165.1 143.51)
+		)
+		(stroke
+			(width 0)
+			(type default)
+		)
+	)
+	(wire
+		(pts
 			(xy 219.71 69.85) (xy 245.11 69.85)
 		)
@@
 	(wire
 		(pts
-			(xy 184.15 147.32) (xy 184.15 138.43)
+			(xy 184.15 147.32) (xy 184.15 139.7)
 		)
 		(stroke
@@
 	(wire
 		(pts
-			(xy 176.53 143.51) (xy 151.13 143.51)
-		)
-		(stroke
-			(width 0)
-			(type default)
-		)
-	)
-	(wire
-		(pts
 			(xy 283.21 44.45) (xy 295.91 44.45)
 		)
@@
 	(wire
 		(pts
-			(xy 151.13 138.43) (xy 184.15 138.43)
-		)
-		(stroke
-			(width 0)
-			(type default)
-		)
-	)
-	(wire
-		(pts
 			(xy 295.91 90.17) (xy 295.91 100.33)
 		)
@@
 	(wire
 		(pts
+			(xy 151.13 138.43) (xy 165.1 138.43)
+		)
+		(stroke
+			(width 0)
+			(type default)
+		)
+	)
+	(wire
+		(pts
 			(xy 351.79 109.22) (xy 351.79 149.86)
 		)
@@
 	(wire
 		(pts
+			(xy 184.15 139.7) (xy 184.15 138.43)
+		)
+		(stroke
+			(width 0)
+			(type default)
+		)
+	)
+	(wire
+		(pts
 			(xy 386.08 104.14) (xy 386.08 95.25)
 		)
@@
 	(wire
 		(pts
-			(xy 176.53 156.21) (xy 176.53 143.51)
+			(xy 176.53 142.24) (xy 176.53 156.21)
 		)
 		(stroke
@@
 					(unit 1)
 				)
+			)
+		)
+	)
+	(symbol
+		(lib_id "Connector:Screw_Terminal_01x02")
+		(at 171.45 139.7 0)
+		(mirror y)
+		(unit 1)
+		(body_style 1)
+		(exclude_from_sim no)
+		(in_bom yes)
+		(on_board yes)
+		(in_pos_files yes)
+		(dnp no)
+		(property "Reference" "J10"
+			(at 168.91 139.6999 0)
+			(show_name no)
+			(do_not_autoplace no)
+			(effects
+				(font
+					(size 1.27 1.27)
+				)
+				(justify left)
+			)
+		)
+		(property "Value" "SMPS_IN"
+			(at 168.91 142.2399 0)
+			(show_name no)
+			(do_not_autoplace no)
+			(effects
+				(font
+					(size 1.27 1.27)
+				)
+				(justify left)
+			)
+		)
+		(property "Footprint" "TerminalBlock_Phoenix:TerminalBlock_Phoenix_MKDS-1,5-2-5.08_1x02_P5.08mm_Horizontal"
+			(at 171.45 139.7 0)
+			(hide yes)
+			(show_name no)
+			(do_not_autoplace no)
+			(effects
+				(font
+					(size 1.27 1.27)
+				)
+			)
+		)
+		(property "Datasheet" "https://www.farnell.com/datasheets/2325533.pdf"
+			(at 171.45 139.7 0)
+			(hide yes)
+			(show_name no)
+			(do_not_autoplace no)
+			(effects
+				(font
+					(size 1.27 1.27)
+				)
+			)
+		)
+		(property "Description" "Generic screw terminal, single row, 01x02, script generated (kicad-library-utils/schlib/autogen/connector/)"
+			(at 171.45 139.7 0)
+			(hide yes)
+			(show_name no)
+			(do_not_autoplace no)
+			(effects
+				(font
+					(size 1.27 1.27)
+				)
+			)
+		)
+		(property "LCSC" "C5443539"
+			(at 171.45 139.7 0)
+			(hide yes)
+			(show_name no)
+			(do_not_autoplace no)
+			(effects
+				(font
+					(size 1.27 1.27)
+				)
+			)
+		)
+		(property "Field5" ""
+			(at 171.45 139.7 0)
+			(hide yes)
+			(show_name no)
+			(do_not_autoplace no)
+			(effects
+				(font
+					(size 1.27 1.27)
+				)
+			)
+		)
+		(pin "2"
+		)
+		(pin "1"
+		)
+		(instances
+			(project "PSU"
+				(path "/fa85d71b-1ddc-4df3-8621-90a970c44e66"
+					(reference "J10")
+					(unit 1)
+				)

Commit message: quick update / fix
Parts:
- U5: value 3v3 Mornsun URB4803LD-20WR3 -> 3v3 Mornsun URB2403LD-20WR3
- U7: value 12v Mornsun URB2412LD-30WR3 -> 12v Mornsun URB2412LD-50WR3; footprint Converter_DCDC:Converter_DCDC_XP_POWER_JTDxxxxxxx_THT -> My Footprints:urb 50w dc-dc
Connections:
- net at C15.2, C22.2, C23.2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: now also U5.2 (GND), U5.6 (GND), U7.2 (GND); no longer U5.3 (GND), U5.5 (0V), U7.3 (GND)
- net at L1.2, R16.1, U6.10 (Vin)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: now also U5.3 (Vin), U7.3 (Vin); no longer U5.2 (Vin), U7.2 (Vin)
Other:
- note added: "COMPONENT NOTES: R1, R2, R3, (discharges big filter caps) use at least 1W at least Resistors. For all other resistors, use 1/4W. All resistors are metal film, 1% or better tolerance. All screw terminals (J2, J3, J4. J5, J9, J10) are the Phoenix Contact MKDS 1,5 series, 5.08mm pin pitch. Pin headers (J6, J7, J8) are standard 2.54mm pin pitch male pin headers. Regulators (U1, U2, U3) are all TO-220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"
- note added: "revision 0.1"
- note removed: "COMPONENT NOTES: R1, R2, R3, (discharges big filter caps) use at least 1W at least Resistors. For all other resistors, use 1/4W. All resistors are metal film, 1% or better tolerance. All screw terminals (J2, J3, J4. J5, J9, J10) are the Phoenix Contact MKDS 1,5 series, 5.08mm pin pitch. Pin headers (J2, J9, J10) are standard 2.54mm pin pitch male pin headers. Regulators (U1, U2, U3) are all TO-22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"
- note removed: "revision 0"

Commit message: did some stuff lol
Parts:
- TR2: value Amgis L01-6320 -> Amgis L01-6330
Changed lines of the file:
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@@
 			)
 		)
-		(property "Value" "Amgis L01-6320"
+		(property "Value" "Amgis L01-6330"
 			(at 194.31 101.6 0)
 			(show_name no)
