File: PCB/CHANNELSTRIP_CONTROLS_CARD/channel.kicad_pcb (KiCad board)
At the start: 2 copper layers, 40 x 480 mm, 54 parts, among them J1 CONN, J18 KNOB_LED_D1, J19 KNOB_LED_D1, J2 SCREEN, J20 KNOB_LED_D1, J21 KNOB_LED_D1, J22 KNOB_LED_P1, J23 KNOB_LED_P1, J24 KNOB_LED_P1, J25 KNOB_LED_P1, J26 KNOB_LED_D1, J27 KNOB_LED_D1, J28 KNOB_LED_P1, J29 KNOB_LED_P1, J30 KNOB_LED_D1, J31 KNOB_LED_D1, J32 KNOB_LED_D1, J33 KNOB_LED_D1, J34 KNOB_LED_P1, J35 KNOB_LED_P1, J36 KNOB_LED_P1, J37 KNOB_LED_P1, SW10 KNOB_CTRL_4A, SW11 LINE, SW12 PHASE, SW13 COMP, SW14 SOLO, SW15 KNOB_INPUT, SW16 KNOB_PAN, SW17 HIZ, SW18 HPF, SW19 SEND, SW20 MUTE, SW21 KNOB_CTRL_1B, SW22 KNOB_CTRL_2B, SW23 KNOB_CTRL_3B, SW24 KNOB_CTRL_4B, SW25 INS, SW26 PRE, SW27 SEL, SW4 MIC, SW5 V48, SW6 EQ, SW7 KNOB_CTRL_1A, SW8 KNOB_CTRL_2A, SW9 KNOB_CTRL_3A, U10 TTP223-BA6, U4 MCP23017x-x-ML, U5 MCP23017x-x-ML, U6 MCP23017x-x-ML, U7 MCP23017x-x-ML, U8 74HCT595D, U9 74HCT595D

Commit message: im cray cray
Parts:
- removed U7: MCP23017x-x-ML, Package_DFN_QFN:QFN-28-1EP_6x6mm_P0.65mm_EP4.25x4.25mm
- added R1: 330, Resistor_SMD:R_0603_1608Metric, F.Cu at (68.5, 179.6)
- added R10: 330, Resistor_SMD:R_0603_1608Metric, F.Cu at (46.4, 370.5)
- added R11: 330, Resistor_SMD:R_0603_1608Metric, F.Cu at (46.4, 372.3)
- added R12: 330, Resistor_SMD:R_0603_1608Metric, F.Cu at (46.4, 374.1)
- added R13: 330, Resistor_SMD:R_0603_1608Metric, F.Cu at (46.4, 375.9)
- added R14: 330, Resistor_SMD:R_0603_1608Metric, F.Cu at (46.4, 377.7)
- added R2: 330, Resistor_SMD:R_0603_1608Metric, F.Cu at (79.9, 183.7)
- added R3: 330, Resistor_SMD:R_0603_1608Metric, F.Cu at (79.9, 181.6)
- added R4: 330, Resistor_SMD:R_0603_1608Metric, F.Cu at (79.9, 179.5)
- added R5: 330, Resistor_SMD:R_0603_1608Metric, F.Cu at (79.9, 177.5)
- added R6: 330, Resistor_SMD:R_0603_1608Metric, F.Cu at (79.9, 175.5)
- added R7: 330, Resistor_SMD:R_0603_1608Metric, F.Cu at (79.9, 173.4)
- added R8: 330, Resistor_SMD:R_0603_1608Metric, F.Cu at (79.9, 171.3)
- added R9: 330, Resistor_SMD:R_0603_1608Metric, F.Cu at (54.9, 369.7)
- J1: moved to B.Cu
- J18, J19, J20, J21, J26, J27, J30, J31, J32, J33: footprint Connector_PinSocket_2.54mm:PinSocket_1x05_P2.54mm_Vertical -> Connector_PinSocket_2.54mm:PinSocket_1x04_P2.54mm_Vertical
- U4, U5, U6: footprint Package_DFN_QFN:QFN-28-1EP_6x6mm_P0.65mm_EP4.25x4.25mm -> Package_DFN_QFN:QFN-28-1EP_6x6mm_P0.65mm_EP4.25x4.25mm_ThermalVias
- moved SW26 440.9 mm to (50.7, 461.7)
- moved SW25 433.5 mm to (50.7, 442.8)
- moved U9 411.0 mm to (51.7, 376.7)
- moved SW20 389.8 mm to (64.0, 390.0)
- moved SW14 379.9 mm to (51.0, 390.0)
- moved U10 372.6 mm to (78.4, 424.5)
- moved J29 357.9 mm to (60.2, 397.7)
- moved SW16 357.9 mm to (64.1, 408.6)
- moved J27 357.7 mm to (60.2, 418.2)
- moved SW27 354.1 mm to (77.0, 390.0)
- moved J1 304.4 mm to (62.7, 380.7)
- moved J2 301.8 mm to (78.1, 352.6), turned to -90 degrees
- moved SW15 297.5 mm to (64.0, 118.2)
- moved J28 296.9 mm to (60.5, 107.3)
- moved J26 296.9 mm to (60.5, 127.8)
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Connections:
- J1 pad 16: DISP_BRIGHT_PWM -> DISP_SPI_MOSI
- J1 pad 18: DISP_SPI_MOSI -> DISP_RST
- J1 pad 20: DISP_SPI_CL -> DISP_TE
- J1 pad 22: DISP_RST -> DISP_CS
- J1 pad 24: DISP_TE -> DISP_SPI_CL
- J1 pad 26: DISP_CS -> DISP_A0
- J1 pad 28: DISP_A0 -> DISP_BRIGHT_PWM
- J22 pad 1: GND -> Net-(J22-Pin_1)
- J23 pad 1: GND -> Net-(J23-Pin_1)
- J24 pad 1: GND -> Net-(J24-Pin_1)
- J25 pad 1: GND -> Net-(J25-Pin_1)
- J28 pad 1: GND -> Net-(J18-Pin_1)
- J29 pad 1: GND -> Net-(J29-Pin_1)
- J30 pad 1: Net-(J18-Pin_5) -> Net-(J22-Pin_1)
- J31 pad 1: Net-(J19-Pin_5) -> Net-(J23-Pin_1)
- J32 pad 1: Net-(J20-Pin_5) -> Net-(J24-Pin_1)
- J33 pad 1: Net-(J21-Pin_5) -> Net-(J25-Pin_1)
- J34 pad 1: GND -> Net-(J19-Pin_1)
- J35 pad 1: GND -> Net-(J20-Pin_1)
- J36 pad 1: GND -> Net-(J21-Pin_1)
- J37 pad 1: GND -> Net-(J27-Pin_1)
- U8 pad 14: Net-(J27-Pin_5) -> Net-(J29-Pin_1)
- U9 pad 6: Net-(U9-QG) -> unconnected-(U9-QG-Pad6)
- U9 pad 7: Net-(U9-QH) -> unconnected-(U9-QH-Pad7)
Routing:
- net +5V: track 0.00 -> 441.5 mm, vias 0 -> 5
- net LED_CL: track 0.00 -> 407.2 mm, vias 0 -> 13
- net LED_LATCH: track 0.00 -> 400.8 mm, vias 0 -> 2
- net LED_BRIGHT_PWM: track 0.00 -> 391.7 mm, vias 0 -> 3
- net +3.3V: track 0.00 -> 351.8 mm, vias 0 -> 16
- net /A14: track 0.00 -> 322.2 mm, vias 0 -> 2
- net /A13: track 0.00 -> 320.0 mm, vias 0 -> 3
- net LED_DA: track 0.00 -> 280.0 mm
- net ADDR_MSB: track 0.00 -> 263.0 mm, vias 0 -> 7
- net /A11: track 0.00 -> 258.1 mm, vias 0 -> 1
- net /A12: track 0.00 -> 254.9 mm, vias 0 -> 1
- net /A10: track 0.00 -> 250.2 mm, vias 0 -> 1
- net /B9: track 0.00 -> 243.8 mm, vias 0 -> 1
- net Net-(J29-Pin_1): track 0.00 -> 234.3 mm, vias 0 -> 1
- net KNOB_I2C_DA: track 0.00 -> 233.2 mm, vias 0 -> 5
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- added copper zone on B.Cu, net GND
- added copper zone on F.Cu, net GND
- added copper zone on In1.Cu, net GND
Other:
- copper layers 2 -> 4
- board text added: "1 2"
- board text added: "31 32"
- board text added: "ANLG_GND 3V3_ANLG_REF DISP_PWM_LITE DISP_A0 DISP_SCL DISP_CS DISP_TE DISP_RST DISP_MOSI +2V8_DISP +2V8_DISP +10V_MOTOR +10V_MOTOR +3V3_DIGI +3V3_DIGI"
- board text added: "INPUT"
- board text added: "KNOB 1A"
- board text added: "KNOB 1B"
- board text added: "KNOB 2A"
- board text added: "KNOB 2B"
- board text added: "KNOB 3A"
- board text added: "KNOB 3B"
- board text added: "KNOB 4A"
- board text added: "KNOB 4B"
- board text added: "LED_CLK"
- board text added: "LED_DA"
- board text added: "LED_LATCH"
- board text added: "LED_PWM_BRITE"
- board text added: "MOT_B_DIR MOT_A_DIR FADER_TOUCH FADER_ADC CTRLS_CLK CTRLS_DA GND GND ADDR_MSB +5V_LEDS +5V_LEDS +5V_LEDS"
- board text added: "OUT_LED_CAS"
- board text added: "PAN"
