File: PCB/CHANNELSTRIP_CONTROLS_CARD/channel.kicad_sch (KiCad schematic)
At the start: 69 parts, among them J1 CONN, J18 KNOB_LED_D1, J19 KNOB_LED_D1, J2 SCREEN, J20 KNOB_LED_D1, J21 KNOB_LED_D1, J22 KNOB_LED_P1, J23 KNOB_LED_P1, J24 KNOB_LED_P1, J25 KNOB_LED_P1, J26 KNOB_LED_D1, J27 KNOB_LED_D1, J28 KNOB_LED_P1, J29 KNOB_LED_P1, J30 KNOB_LED_D1, J31 KNOB_LED_D1, J32 KNOB_LED_D1, J33 KNOB_LED_D1, J34 KNOB_LED_P1, J35 KNOB_LED_P1, J36 KNOB_LED_P1, J37 KNOB_LED_P1, SW10 KNOB_CTRL_4A, SW11 LINE, SW12 PHASE, SW13 COMP, SW14 SOLO, SW15 KNOB_INPUT, SW16 KNOB_PAN, SW17 HIZ, SW18 HPF, SW19 SEND, SW20 MUTE, SW21 KNOB_CTRL_1B, SW22 KNOB_CTRL_2B, SW23 KNOB_CTRL_3B, SW24 KNOB_CTRL_4B, SW25 INS, SW26 PRE, SW27 SEL, SW4 MIC, SW5 V48, SW6 EQ, SW7 KNOB_CTRL_1A, SW8 KNOB_CTRL_2A, SW9 KNOB_CTRL_3A, U10 TTP223-BA6, U4 MCP23017x-x-ML, U5 MCP23017x-x-ML, U6 MCP23017x-x-ML, U8 74HCT595D, U9 74HCT595D

Commit message: im cray cray
Parts:
- removed R15, R16: 330, symbol Device:R_US
- F1, J1, SW10, SW11, SW12, SW13, SW14, SW15, SW16, SW17, SW18, SW19, SW20, SW21, SW22, SW23, SW24, SW25, SW26, SW27, SW4, SW5, SW6, SW7, SW8, SW9: now not fitted
- J18, J19, J20, J21, J26, J27, J30, J31, J32, J33: footprint Connector_PinSocket_2.54mm:PinSocket_1x05_P2.54mm_Vertical -> Connector_PinSocket_2.54mm:PinSocket_1x04_P2.54mm_Vertical; symbol Connector:Conn_01x05_Pin -> Connector:Conn_01x04_Pin; LCSC (none) -> C2718488
- J2: LCSC (none) -> C22435644
- J22, J23, J24, J25, J28, J29, J34, J35, J36, J37: LCSC (none) -> C2718488
- R1, R10, R11, R12, R13, R14, R2, R3, R4, R5, R6, R7, R8, R9: footprint (none) -> Resistor_SMD:R_0603_1608Metric; LCSC (none) -> C25231
- U10: LCSC (none) -> C42422127
- U4, U5, U6: footprint Package_DFN_QFN:QFN-28-1EP_6x6mm_P0.65mm_EP4.25x4.25mm -> Package_DFN_QFN:QFN-28-1EP_6x6mm_P0.65mm_EP4.25x4.25mm_ThermalVias; LCSC (none) -> C629439
Connections:
- net DISP_A0: now also J1.26 (Pin_26); no longer J1.28 (Pin_28)
- net DISP_BRIGHT_PWM: now also J1.28 (Pin_28); no longer J1.16 (Pin_16)
- net DISP_CS: now also J1.22 (Pin_22); no longer J1.26 (Pin_26)
- net DISP_RST: now also J1.18 (Pin_18); no longer J1.22 (Pin_22)
- net DISP_SPI_CL: now also J1.24 (Pin_24); no longer J1.20 (Pin_20)
- net DISP_SPI_MOSI: now also J1.16 (Pin_16); no longer J1.18 (Pin_18)
- net DISP_TE: now also J1.20 (Pin_20); no longer J1.24 (Pin_24)
- net GND: no longer J22.1 (Pin_1), J23.1 (Pin_1), J24.1 (Pin_1), J25.1 (Pin_1), J28.1 (Pin_1), J29.1 (Pin_1), J34.1 (Pin_1), J35.1 (Pin_1), J36.1 (Pin_1), J37.1 (Pin_1)
- net at J18.1 (Pin_1): now also J28.1 (Pin_1); no longer J26.5 (Pin_5)
- net at J31.1 (Pin_1): now also J23.1 (Pin_1); no longer J19.5 (Pin_5)
- net at J20.1 (Pin_1): now also J35.1 (Pin_1); no longer J31.5 (Pin_5)
- net at J30.1 (Pin_1): now also J22.1 (Pin_1); no longer J18.5 (Pin_5)
- net at U8.14 (SER): now also J29.1 (Pin_1); no longer J27.5 (Pin_5)
- net at J32.1 (Pin_1): now also J24.1 (Pin_1); no longer J20.5 (Pin_5)
- net at J19.1 (Pin_1): now also J34.1 (Pin_1); no longer J30.5 (Pin_5)
- net at J27.1 (Pin_1): now also J37.1 (Pin_1); no longer J33.5 (Pin_5)
- net at J33.1 (Pin_1): now also J25.1 (Pin_1); no longer J21.5 (Pin_5)
- net at J21.1 (Pin_1): now also J36.1 (Pin_1); no longer J32.5 (Pin_5)
- no-connect marks 8 -> 10
