File: PCB/led_ring_knob/kicad project/led_ring.kicad_sch (KiCad schematic)
At the start: 70 parts, among them J1 DATA, J2 POW, U1 74HCT595PW, U2 74HCT595PW, U3 74HCT595PW, U4 74HCT595PW

Commit message: led ring redesign
Parts:
- D1, D10, D11, D12, D13, D14, D15, D16, D17, D18, D19, D2, D20, D21, D22, D23, D24, D25, D26, D27, D28, D29, D3, D30, D31, D32, D4, D5, D6, D7, D8, D9: LCSC C6768746 -> C52675959
- J1: footprint Connector_PinHeader_2.54mm:PinHeader_1x05_P2.54mm_Vertical -> Connector_PinHeader_2.54mm:PinHeader_1x04_P2.54mm_Vertical; symbol Connector:Conn_01x05_Pin -> Connector:Conn_01x04_Pin
- R1, R10, R11, R12, R13, R14, R15, R16, R17, R18, R19, R2, R20, R21, R22, R23, R24, R25, R26, R27, R28, R29, R3, R30, R31, R32, R4, R5, R6, R7, R8, R9: value 330 -> 470; LCSC (none) -> C295802
Connections:
- net at D1.1 (K), D10.1 (K), D11.1 (K)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: no longer J2.1 (Pin_1)
- net at U4.9 (QH'): now also J2.1 (Pin_1); no longer J1.5 (Pin_5)
Other:
- note added: "POW: 1 = SERIAL OUT (CASCADE) 2 = GND 3 = 5V 4 = 5V"
- note removed: "POW: 1 = GND 2 = GND 3 = 5V 4 = 5V"

Commit message: im cray cray
Other:
- note added: "DATA: 1 = SERIAL IN 2 = CLK 3 = LATCH ENABLE 4 = OUTPUT ENABLE"
- note removed: "DATA: 1 = SERIAL IN 2 = CLK 3 = LATCH ENABLE 4 = OUTPUT ENABLE 5 = SERIAL OUT (Cascade)"
Changed lines of the file:
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@@
 	(generator_version "10.0")
 	(paper "A4")
-	(text "DATA:\n1 = SERIAL IN\n2 = CLK\n3 = LATCH ENABLE\n4 = OUTPUT ENABLE\n5 = SERIAL OUT (Cascade)"
+	(text "DATA:\n1 = SERIAL IN\n2 = CLK\n3 = LATCH ENABLE\n4 = OUTPUT ENABLE"
 		(exclude_from_sim no)
 		(at 53.086 49.784 0)
